Commit message: Ran poetry and saved command so I can remember it on home computer

File: iiwa_batter/assets/iiwa14_limitless.urdf (robot description, URDF)
Before this commit: robot iiwa14, 11 links, 10 joints
Joints:
- joint iiwa_joint_1: limit lower=-2.96705972839 upper=2.96705972839 -> (none)
- joint iiwa_joint_2: limit lower=-2.09439510239 upper=2.09439510239 effort=320 velocity=1.4835298641951802 -> (none)
- joint iiwa_joint_3: limit lower=-2.96705972839 upper=2.96705972839 effort=176 velocity=1.7453292519943295 -> (none)
- joint iiwa_joint_4: limit lower=-2.09439510239 upper=2.09439510239 effort=176 velocity=1.3089969389957472 -> (none)
- joint iiwa_joint_5: limit lower=-2.96705972839 upper=2.96705972839 effort=110 velocity=2.2689280275926285 -> (none)
- joint iiwa_joint_6: limit lower=-2.09439510239 upper=2.09439510239 effort=40 velocity=2.356194490192345 -> (none)
- joint iiwa_joint_7: limit lower=-3.05432619099 upper=3.05432619099 effort=40 velocity=2.356194490192345 -> (none)
