Commit message: human machine learned the kr6r900, slight refactoring to make it easier to do this process by hand

File: iiwa_batter/assets/kr6r900.urdf (robot description, URDF)
Before this commit: robot iiwa14, 11 links, 10 joints
Joints:
- joint iiwa_joint_3: limit lower=0 upper=0 effort=176 velocity=1.7453292519943295 -> lower=0 upper=0 effort=176 velocity=0
